Commit message: Collision added

File: my_robot_description/urdf/common_properties.urdf.xacro (robot description, xacro)
@@ -1,4 +1,5 @@
 <?xml version="1.0"?>
 <robot xmlns:xacro="https://www.ros.org/wiki/xacro">
+    <!-- ==================== Inertial Macros ==================== -->
     <xacro:macro name="box_inertia" params="m x y z o_xyz o_rpy">
         <inertial>

File: my_robot_description/urdf/my_robot.urdf.xacro (robot description, xacro)
@@ -19,4 +19,10 @@
                 <material name="flange_steel"/>
             </visual>
+            <collision>
+                <geometry>
+                    <sphere radius="${wheel_radius}"/>
+                </geometry>
+                <origin xyz="0 0 0" rpy="0 0 0"/>
+            </collision>
             <xacro:cylinder_inertia m="1.0" r="${wheel_radius}" l="${wheel_length}" o_xyz="0 0 0" o_rpy="${pi/2.0} 0 0" />
         </link>
@@ -32,4 +38,10 @@
             <material name="blue"/>
         </visual>
+        <collision>
+            <geometry>
+                <box size="${base_length} ${base_width} ${base_height}"/>
+            </geometry>
+            <origin xyz="0 0 ${base_height/2}" rpy="0 0 0"/>
+        </collision>
         <xacro:box_inertia m="5.0" x="${base_length}" y="${base_width}" z="${base_height}" o_xyz="0 0 ${base_height/2}" o_rpy="0 0 0" />
     </link>
@@ -67,4 +79,10 @@
             <material name="flange_steel"/>
         </visual>
+        <collision>
+            <geometry>
+                <sphere radius="${front_wheel_radius}"/>
+            </geometry>
+            <origin xyz="0 0 0" rpy="0 0 0"/>
+        </collision>
         <xacro:sphere_inertia m="0.5" r="${front_wheel_radius}" o_xyz="0 0 0" o_rpy="0 0 0" />
     </link>
