Commit message: Issues Fix, ROS_GZ Bridge add

File: my_robot_description/urdf/my_robot.urdf.xacro (robot description, xacro)
@@ -1,5 +1,4 @@
 <?xml version="1.0"?>
 <robot  xmlns:xacro="https://www.ros.org/wiki/xacro">
-    <!-- ==================== Materials ==================== -->
     <!-- ==================== Veriables ==================== -->
     <xacro:property name="base_length" value="0.9"/>
@@ -88,9 +87,8 @@
     </link>
     <!-- Base to front Wheel Joint -->
-    <joint name="base_front_wheel_joint" type="continuous">
+    <joint name="base_front_wheel_joint" type="fixed">
         <parent link="base_link"/>
         <child link="front_wheel"/>
         <origin xyz="${base_length/3.0} 0 ${-front_wheel_radius}" rpy="0 0 0"/>
-        <axis xyz="0 1 0"/>
     </joint>
 </robot>

File: my_robot_description/urdf/robot_complete.urdf.xacro (robot description, xacro)
@@ -4,3 +4,4 @@
     <xacro:include filename="common_properties.urdf.xacro"/>
     <xacro:include filename="my_robot.urdf.xacro"/>
+    <xacro:include filename="my_robot_gazebo_setup.xacro"/>
 </robot>
