Commit message: camera adjusted for OpenCV

File: my_robot_description/urdf/my_robot_camera.xacro (robot description, xacro)
@@ -23,4 +23,10 @@
         <origin xyz ="${(base_length + camera_length)/2.0} 0 ${base_height/2.0}" rpy ="0 0 0"/>
     </joint>
+    <link name="camera_link_optical" />
+    <joint name="camera_optical_joint" type="fixed">
+        <origin xyz="0 0 0" rpy="${-pi/2} 0 ${-pi/2}"/>
+        <parent link="camera_link"/>
+        <child link="camera_link_optical"/>
+    </joint>
     <gazebo reference="camera_link">
         <sensor name="camera" type="camera">
@@ -41,5 +47,5 @@
                     <stddev>0.007</stddev>
                 </noise>
-                <optical_frame_id>camera_link</optical_frame_id>
+                <optical_frame_id>camera_link_optical</optical_frame_id>
                 <camera_info_topic>camera/camera_info</camera_info_topic>
             </camera>
